Commit message: modified urdf but needs work

File: src/f1tenth_stack/urdf/f110.urdf (robot description, URDF)
Before this commit: robot AV21, 19 links, 18 joints
Links:
- removed link camera_front_1
- removed link camera_front_2
- removed link camera_front_left
- removed link camera_front_right
- removed link camera_rear_left
- removed link camera_rear_right
- removed link gps_bottom
- removed link gps_top
- removed link luminar_front
- removed link luminar_left
- removed link luminar_right
- removed link radar_front
- removed link radar_port
- removed link radar_rear
- removed link radar_starboard
- link rear_axle_middle_ground: geometry 
Joints:
- removed joint camera_front_1_joint
- removed joint camera_front_2_joint
- removed joint camera_front_left_joint
- removed joint camera_front_right_joint
- removed joint camera_rear_left_joint
- removed joint camera_rear_right_joint
- removed joint gps_bottom_joint
- removed joint gps_top_joint
- removed joint luminar_front_joint
- removed joint luminar_left_joint
- removed joint luminar_right_joint
- removed joint radar_front_joint
- removed joint radar_port_joint
- removed joint radar_rear_joint
- removed joint radar_starboard_joint

Commit message: updated urdf

File: src/f1tenth_stack/urdf/f110.urdf (robot description, URDF)
Before this commit: robot f110, 4 links, 3 joints
Links:
- added link lidar_link
Joints:
- added joint lidar_joint: type fixed, parent rear_axle_middle, child lidar_link, origin xyz=0.06 0.0 0.185
- joint imu_joint: origin xyz=1.606 0.0 -0.0703 -> xyz=0.15 -0.06 0.05
- joint rear_axle_middle_ground_joint: origin xyz=0 0 -0.198 -> xyz=0 0 -0.05
- joint rear_axle_middle_joint: origin xyz=-1.3206 0.030188 -0.23598 -> xyz=-0.13 0.0 -0.02

Commit message: updated lidar link

File: src/f1tenth_stack/urdf/f110.urdf (robot description, URDF)
Before this commit: robot f110, 5 links, 4 joints
Links:
- removed link lidar_link
- added link laser
Joints:
- joint lidar_joint: child lidar_link -> laser

Commit message: added odom to urdf

File: src/f1tenth_stack/urdf/f110.urdf (robot description, URDF)
Before this commit: robot f110, 5 links, 4 joints
Links:
- added link vesc_odom
Joints:
- added joint vesc_odom_joint: type fixed, parent rear_axle_middle, child vesc_odom, origin xyz=0.15 -0.06 0.05

Commit message: added ekf to stack

File: src/f1tenth_stack/urdf/f110.urdf (robot description, URDF)
Before this commit: robot f110, 6 links, 5 joints
Links:
- removed link center_of_gravity
- removed link vesc_odom
- added link base_link
Joints:
- removed joint vesc_odom_joint
- joint rear_axle_middle_joint: parent center_of_gravity -> base_link
